File: Unisonic21.sch (KiCad schematic (older format))
At the start: 0 parts

Commit message: Adds clock phase generator schematics and PDFs, adds generic gates to mos.lib
Connections:
- wire segments 20 -> 18
Changed lines of the file:
@@
 $Descr A4 11693 8268
 encoding utf-8
-Sheet 1 7
+Sheet 1 8
 Title ""
 Date ""
@@
 PIN2_A
 Wire Wire Line
-	5200 1250 5500 1250
-Wire Wire Line
-	5500 1250 5750 1250
+	5200 1250 5750 1250
 $Sheet
 S 5750 1900 850  550
@@
 	5200 1400 5600 1400
 Wire Wire Line
-	5600 1400 5600 2050
-Wire Wire Line
-	5600 2050 5600 2850
+	5600 1400 5600 2850
 Wire Wire Line
 	5600 2050 5750 2050
